File: kicad/NerdEKO-Gamma-NoATX.kicad_sch (KiCad schematic)
At the start: 24 parts, among them J1 Conn_01x02, J3 Conn_01x01, J5 Conn_01x01

Commit message: final update
Version 1.0 : working as expected, 14TH/s
Parts:
- C1: P/N LCSC (none) -> C2980548
- D1: P/N LCSC (none) -> C913075
- J1: P/N LCSC (none) -> C7426780
- R16: P/N LCSC (none) -> C17513
Changed lines of the file:
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@@
+			)
+		)
+		(property "P/N LCSC" "C17513"
+			(at 64.77 63.5 0)
+			(effects
+				(font
+					(size 1.27 1.27)
+				)
+				(hide yes)
 			)
 		)
@@
 		)
 		(property "P/N MOUSER" "859-LTST-C171GKT"
+			(at 64.77 55.88 0)
+			(effects
+				(font
+					(size 1.27 1.27)
+				)
+				(hide yes)
+			)
+		)
+		(property "P/N LCSC" "C913075"
 			(at 64.77 55.88 0)
 			(effects
@@
 			)
 		)
+		(property "P/N LCSC" "C7426780"
+			(at 26.67 77.47 0)
+			(effects
+				(font
+					(size 1.27 1.27)
+				)
+				(hide yes)
+			)
+		)
 		(pin "1"
 		)
@@
 			(at 43.18 62.23 0)
 			(effects
+				(font
+					(size 1.27 1.27)
+				)
+				(hide yes)
+			)
+		)
+		(property "P/N LCSC" "C2980548"
+			(at 43.18 62.23 0)
+			(effects
