File: kicad/PowerStage.kicad_sch (KiCad schematic)
At the start: 12 parts, among them U19 CSD95472Q5MC

Commit message: final update
Version 1.0 : working as expected, 14TH/s
Parts:
- C177, C179, C318: P/N LCSC (none) -> C476766
- C178: P/N LCSC (none) -> C5448893
- C180, C181: P/N LCSC (none) -> C106244
- C25: P/N LCSC (none) -> C52306
- C319: P/N LCSC (none) -> C344171
- L5: P/N LCSC (none) -> C2639748
- R48, R49: P/N LCSC (none) -> C163970
- U19: P/N LCSC (none) -> C1880674
Changed lines of the file:
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@@
+			)
+		)
+		(property "P/N LCSC" "C106244"
+			(at 167.64 113.03 0)
+			(effects
+				(font
+					(size 1.27 1.27)
+				)
+				(hide yes)
 			)
 		)
@@
 			)
 		)
+		(property "P/N LCSC" "C163970"
+			(at 111.76 90.17 0)
+			(effects
+				(font
+					(size 1.27 1.27)
+				)
+				(hide yes)
+			)
+		)
 		(pin "1"
 		)
@@
 			)
 		)
+		(property "P/N LCSC" "C163970"
+			(at 167.64 104.14 0)
+			(effects
+				(font
+					(size 1.27 1.27)
+				)
+				(hide yes)
+			)
+		)
 		(pin "1"
 		)
@@
 		)
 		(property "Puissance" ""
+			(at 86.36 62.23 0)
+			(effects
+				(font
+					(size 1.27 1.27)
+				)
+				(hide yes)
+			)
+		)
+		(property "P/N LCSC" "C344171"
 			(at 86.36 62.23 0)
 			(effects
@@
 		)
 		(property "Puissance" ""
+			(at 93.98 39.37 0)
+			(effects
+				(font
+					(size 1.27 1.27)
+				)
+				(hide yes)
+			)
+		)
+		(property "P/N LCSC" "C106244"
 			(at 93.98 39.37 0)
 			(effects
@@
 			)
 		)
+		(property "P/N LCSC" "C5448893"
+			(at 120.65 111.76 0)
+			(effects
+				(font
+					(size 1.27 1.27)
+				)
+				(hide yes)
+			)
+		)
 		(pin "2"
 		)
@@
 		)
 		(property "Puissance" ""
+			(at 137.16 90.17 0)
+			(effects
+				(font
+					(size 1.27 1.27)
+				)
+				(hide yes)
+			)
+		)
+		(property "P/N LCSC" "C1880674"
 			(at 137.16 90.17 0)
 			(effects
@@
 			)
 		)
+		(property "P/N LCSC" "C52306"
+			(at 77.47 62.23 0)
+			(effects
+				(font
+					(size 1.27 1.27)
+				)
+				(hide yes)
+			)
+		)
 		(pin "1"
 		)
@@
 			)
 		)
+		(property "P/N LCSC" "C476766"
+			(at 152.4 83.82 0)
+			(effects
+				(font
+					(size 1.27 1.27)
+				)
+				(hide yes)
+			)
+		)
 		(pin "1"
 		)
@@
 		)
 		(property "Puissance" ""
+			(at 186.69 93.98 0)
+			(effects
+				(font
+					(size 1.27 1.27)
+				)
+				(hide yes)
+			)
+		)
+		(property "P/N LCSC" "C2639748"
 			(at 186.69 93.98 0)
 			(effects
@@
 		)
 		(property "Puissance" ""
+			(at 102.87 111.76 0)
+			(effects
+				(font
+					(size 1.27 1.27)
+				)
+				(hide yes)
+			)
+		)
+		(property "P/N LCSC" "C476766"
 			(at 102.87 111.76 0)
 			(effects
@@
 			(at 95.25 62.23 0)
 			(effects
+				(font
+					(size 1.27 1.27)
+				)
+				(hide yes)
+			)
+		)
+		(property "P/N LCSC" "C476766"
+			(at 95.25 62.23 0)
+			(effects
